File: KiCAD Files/CondenserMicAudioDetector/CondenserMicAudioDetector.kicad_pcb (KiCad board)
At the start: 2 copper layers, 50.8 x 40.6 mm, 29 parts, among them Q1 BC547, Q2 BC547, Q3 BC547, Q4 BC557

Commit message: Updated Schematic & PCB Design
Parts:
- added R15: 2k2, Resistor_SMD:R_0805_2012Metric_Pad1.20x1.40mm_HandSolder, B.Cu at (123.2, 91.4)
- added R16: 2k, Resistor_SMD:R_0805_2012Metric_Pad1.20x1.40mm_HandSolder, B.Cu at (120.7, 91.4)
- C1: value 100n -> 1u
- moved R1 3.06 mm to (118.1, 88.9)
Connections:
- R1 pad 2: Net-(MK1-+) -> Net-(R1-Pad2)
Routing:
- net Net-(R1-Pad2): track 0.00 -> 5.30 mm
- net Net-(C4-Pad1): track 58.4 -> 53.8 mm
- net Net-(C2-Pad1): track 24.3 -> 23.5 mm

Commit message: Updated Schematic & PCB
Parts:
- removed R15: 2k2, Resistor_SMD:R_0805_2012Metric_Pad1.20x1.40mm_HandSolder
- R1: value 10k -> 1k8
- moved R1 4.58 mm to (121.9, 91.4)
- moved R16 2.54 mm to (118.1, 91.4)
Connections:
- R1 pad 2: Net-(R1-Pad2) -> Net-(MK1-+)
- R16 pad 1: Net-(R1-Pad2) -> Net-(MK1-+)
Routing:
- net Net-(R1-Pad2): track 5.30 -> 0.00 mm
- net Net-(MK1-+): track 12.5 -> 8.42 mm
- net Net-(C4-Pad1): track 53.8 -> 52.0 mm
- net Net-(Q1-C): track 23.6 -> 22.1 mm
- net Net-(C2-Pad1): track 23.5 -> 22.8 mm
