File: KiCAD Files/CondenserMicAudioDetector/CondenserMicAudioDetector.kicad_sch (KiCad schematic)
At the start: 29 parts, among them Q1 BC547, Q2 BC547, Q3 BC547, Q4 BC557

Commit message: Updated Schematic & PCB Design
Parts:
- added R15: 2k2, Resistor_SMD:R_0805_2012Metric_Pad1.20x1.40mm_HandSolder, symbol Device:R_Small
- added R16: 2k, Resistor_SMD:R_0805_2012Metric_Pad1.20x1.40mm_HandSolder, symbol Device:R_Small
- C1: value 100n -> 1u
Connections:
- net GND: now also R16.2
- net at C1.1, MK1.2 (+): now also R15.1; no longer R1.2
- new net: R1.2, R15.2, R16.1
Other:
- moved on the sheet: MK1, R1, R14, R3, R4, R6, R7

Commit message: Updated Schematic & PCB
Parts:
- removed R15: 2k2, Resistor_SMD:R_0805_2012Metric_Pad1.20x1.40mm_HandSolder, symbol Device:R_Small
- R1: value 10k -> 1k8
Connections:
- net at C1.1, MK1.2 (+): now also R1.2, R16.1
Other:
- moved on the sheet: R1, R16
Changed lines of the file:
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@@
+	)
+	(junction
+		(at 59.69 96.52)
+		(diameter 0)
+		(color 0 0 0 0)
 	)
 	(junction
@@
 	)
 	(junction
-		(at 72.39 96.52)
+		(at 160.02 96.52)
 		(diameter 0)
 		(color 0 0 0 0)
 	)
 	(junction
-		(at 160.02 96.52)
+		(at 72.39 96.52)
 		(diameter 0)
 		(color 0 0 0 0)
@@
 	)
 	(junction
-		(at 72.39 105.41)
-		(diameter 0)
-		(color 0 0 0 0)
-	)
-	(junction
 		(at 87.63 113.03)
 		(diameter 0)
@@
 	(wire
 		(pts
-			(xy 72.39 104.14) (xy 72.39 105.41)
-		)
-		(stroke
-			(width 0)
-			(type default)
-		)
-	)
-	(wire
-		(pts
 			(xy 184.15 76.2) (xy 200.66 76.2)
 		)
@@
 	(wire
 		(pts
-			(xy 72.39 111.76) (xy 72.39 113.03)
+			(xy 72.39 107.95) (xy 72.39 113.03)
 		)
 		(stroke
@@
 	(wire
 		(pts
-			(xy 69.85 92.71) (xy 69.85 105.41)
-		)
-		(stroke
-			(width 0)
-			(type default)
-		)
-	)
-	(wire
-		(pts
 			(xy 184.15 76.2) (xy 184.15 77.47)
 		)
@@
 	(wire
 		(pts
-			(xy 72.39 96.52) (xy 72.39 99.06)
-		)
-		(stroke
-			(width 0)
-			(type default)
-		)
-	)
-	(wire
-		(pts
 			(xy 160.02 88.9) (xy 160.02 96.52)
 		)
@@
 	(wire
 		(pts
+			(xy 72.39 96.52) (xy 78.74 96.52)
+		)
+		(stroke
+			(width 0)
+			(type default)
+		)
+	)
+	(wire
+		(pts
 			(xy 127 96.52) (xy 127 102.87)
 		)
@@
 	(wire
 		(pts
+			(xy 72.39 96.52) (xy 72.39 102.87)
+		)
+		(stroke
+			(width 0)
+			(type default)
+		)
+	)
+	(wire
+		(pts
 			(xy 171.45 85.09) (xy 171.45 86.36)
 		)
@@
 	(wire
 		(pts
+			(xy 59.69 88.9) (xy 59.69 96.52)
+		)
+		(stroke
+			(width 0)
+			(type default)
+		)
+	)
+	(wire
+		(pts
 			(xy 200.66 88.9) (xy 200.66 90.17)
 		)
@@
 	(wire
 		(pts
-			(xy 69.85 105.41) (xy 72.39 105.41)
-		)
-		(stroke
-			(width 0)
-			(type default)
-		)
-	)
-	(wire
-		(pts
 			(xy 87.63 107.95) (xy 87.63 113.03)
 		)
@@
 	(wire
 		(pts
-			(xy 72.39 105.41) (xy 72.39 106.68)
-		)
-		(stroke
-			(width 0)
-			(type default)
-		)
-	)
-	(wire
-		(pts
 			(xy 214.63 76.2) (xy 200.66 76.2)
 		)
@@
 	(wire
 		(pts
-			(xy 72.39 96.52) (xy 78.74 96.52)
-		)
-		(stroke
-			(width 0)
-			(type default)
-		)
-	)
-	(wire
-		(pts
 			(xy 171.45 76.2) (xy 176.53 76.2)
 		)
@@
 	(wire
 		(pts
-			(xy 69.85 76.2) (xy 105.41 76.2)
+			(xy 59.69 76.2) (xy 105.41 76.2)
 		)
 		(stroke
@@
 	(wire
 		(pts
-			(xy 69.85 76.2) (xy 69.85 87.63)
+			(xy 59.69 76.2) (xy 59.69 83.82)
 		)
 		(stroke
@@
 	(symbol
 		(lib_id "Device:R_Small")
-		(at 72.39 101.6 0)
-		(unit 1)
-		(exclude_from_sim no)
-		(in_bom yes)
-		(on_board yes)
-		(dnp no)
-		(fields_autoplaced yes)
-		(property "Reference" "R15"
-			(at 74.93 100.3299 0)
-			(effects
-				(font
-					(size 1.016 1.016)
-				)
-				(justify left)
-			)
-		)
-		(property "Value" "2k2"
-			(at 74.93 102.8699 0)
-			(effects
-				(font
-					(size 1.27 1.27)
-				)
-				(justify left)
-			)
-		)
-		(property "Footprint" "Resistor_SMD:R_0805_2012Metric_Pad1.20x1.40mm_HandSolder"
-			(at 72.39 101.6 0)
-			(effects
-				(font
-					(size 1.27 1.27)
-				)
-				(hide yes)
-			)
-		)
-		(property "Datasheet" "~"
-			(at 72.39 101.6 0)
-			(effects
-				(font
-					(size 1.27 1.27)
-				)
-				(hide yes)
-			)
-		)
-		(property "Description" "Resistor, small symbol"
-			(at 72.39 101.6 0)
-			(effects
-				(font
-					(size 1.27 1.27)
-				)
-				(hide yes)
-			)
-		)
-		(pin "1"
-		)
-		(pin "2"
-		)
-		(instances
-			(project "CondenserMicAudioDetector"
-				(path "/f7756d24-9ca6-4005-8809-37e3ac643dac"
-					(reference "R15")
-					(unit 1)
-				)
-			)
-		)
-	)
-	(symbol
-		(lib_id "Device:R_Small")
 		(at 87.63 90.17 0)
 		(unit 1)
@@
 	(symbol
 		(lib_id "Device:R_Small")
-		(at 69.85 90.17 0)
+		(at 59.69 86.36 0)
 		(unit 1)
 		(exclude_from_sim no)
@@
 		(fields_autoplaced yes)
 		(property "Reference" "R1"
-			(at 72.39 88.8999 0)
+			(at 62.23 85.0899 0)
 			(effects
 				(font
@@
 			)
 		)
-		(property "Value" "10k"
-			(at 72.39 91.4399 0)
+		(property "Value" "1k8"
+			(at 62.23 87.6299 0)
 			(effects
 				(font
@@
 		)
 		(property "Footprint" "Resistor_SMD:R_0805_2012Metric_Pad1.20x1.40mm_HandSolder"
-			(at 69.85 90.17 0)
+			(at 59.69 86.36 0)
 			(effects
 				(font
@@
 		)
 		(property "Datasheet" "~"
-			(at 69.85 90.17 0)
+			(at 59.69 86.36 0)
 			(effects
 				(font
@@
 		)
 		(property "Description" "Resistor, small symbol"
-			(at 69.85 90.17 0)
+			(at 59.69 86.36 0)
 			(effects
 				(font
@@
 	(symbol
 		(lib_id "Device:R_Small")
-		(at 72.39 109.22 0)
+		(at 72.39 105.41 0)
 		(unit 1)
 		(exclude_from_sim no)
@@
 		(fields_autoplaced yes)
 		(property "Reference" "R16"
-			(at 74.93 107.9499 0)
+			(at 74.93 104.1399 0)
 			(effects
 				(font
@@
 		)
 		(property "Value" "2k"
-			(at 74.93 110.4899 0)
+			(at 74.93 106.6799 0)
 			(effects
 				(font
@@
 		)
 		(property "Footprint" "Resistor_SMD:R_0805_2012Metric_Pad1.20x1.40mm_HandSolder"
-			(at 72.39 109.22 0)
+			(at 72.39 105.41 0)
 			(effects
 				(font
@@
 		)
 		(property "Datasheet" "~"
-			(at 72.39 109.22 0)
+			(at 72.39 105.41 0)
 			(effects
 				(font
@@
 		)
 		(property "Description" "Resistor, small symbol"
-			(at 72.39 109.22 0)
-			(effects
-				(font
+			(at 72.39 105.41 0)
+			(effects
+				(font
